File: business-card.sch (KiCad schematic (older format))
At the start: 45 parts, among them J1 Conn_02x04_Counter_Clockwise, J3 USB_B, Q1 Q_NMOS_GSD, SW1 SW_Push, U4 JW5211, U5 JW5211, U6 JW5211, U7 F1C100s, U8 AT25SF081-SSHD-X, Y1 24MHz

Commit message: Remove traces to try autoroute
Parts:
- Y1: symbol Device:Crystal_GND24_Small -> business-card-rescue:Crystal_GND24_Small-Device
Changed lines of the file:
@@
 EESchema Schematic File Version 4
-LIBS:business-card-cache
-EELAYER 26 0
+EELAYER 30 0
 EELAYER END
 $Descr A4 11693 8268
@@
 Connection ~ 9925 1250
 $Comp
-L Device:Crystal_GND24_Small Y1
+L business-card-rescue:Crystal_GND24_Small-Device Y1
 U 1 1 5FCAB95B
 P 10050 1250

Commit message: cleanup
Parts:
- added J2: Conn_02x04_Counter_Clockwise, footprints:SOIC_clipProgSmall, symbol Connector_Generic:Conn_02x04_Counter_Clockwise
Connections:
- net GND: now also J2.5 (Pin_5)
- net SDA: now reaches U7.37 (PE12/DA_MCLK/TWI0_SDA/PWM0/EINTE12)
- net SDA: now also J2.8 (Pin_8)
- net SCL: now reaches U7.38 (PE11/CLK_OUT/TWI0_SCK/IR_RX/EINTE11)
- net SCL: now also J2.1 (Pin_1)
- net JTAG_TCK: now reaches U7.53 (PF5/SDC0_D2/DBG_CK/PWM1/EINTF5)
- net JTAG_TCK: now also J2.6 (Pin_6)
- net JTAG_TMS: now reaches U7.55 (PF3/SDC0_CMD/DBG_DO/EINTF3)
- net JTAG_TMS: now also U7.58 (PF0/SDC0_D1/DBG_MS/IR_RX/EINTF0), J2.2 (Pin_2)
- net JTAG_TDI: now reaches U7.57 (PF1/SDC0_D0/DBG_DI/EINTF1)
- net JTAG_TDI: now also J2.7 (Pin_7)
- new net JTAG_TDO: J2.3 (Pin_3)
- no-connect marks 49 -> 44
Changed lines of the file:
@@
 EESchema Schematic File Version 4
-EELAYER 30 0
+LIBS:business-card-cache
+EELAYER 26 0
 EELAYER END
 $Descr A4 11693 8268
@@
 F 3 "~" H 1150 7300 50  0001 C CNN
 	1    1150 7300
-	1    0    0    -1
-$EndComp
-$Comp
-L business-card-rescue:F1C100s-3340_kicad-business-card-rescue U7
-U 1 1 5FC1F3CA
-P 7050 3250
-F 0 "U7" H 7100 5415 50  0000 C CNN
-F 1 "F1C100s" H 7100 5324 50  0000 C CNN
-F 2 "footprints:QFN-88_EP_10x10_Pitch0.4mm" H 4950 4950 50  0001 C CNN
-F 3 "" H 4950 4950 50  0001 C CNN
-	1    7050 3250
 	1    0    0    -1
 $EndComp
@@
 Wire Wire Line
 	10175 1250 10400 1250
-Wire Wire Line
-	9250 3950 9250 4050
-Connection ~ 9250 4050
-Wire Wire Line
-	9250 4050 9250 4150
-Connection ~ 9250 4150
-Wire Wire Line
-	9250 4150 9250 4250
 $Comp
 L business-card-rescue:power_GND-business-card-cache #PWR0125
@@
 	0    -1   -1   0
 $EndComp
-Connection ~ 9250 4250
 $Comp
 L business-card-rescue:power_GND-business-card-cache #PWR0126
@@
 	0    -1   -1   0
 $EndComp
-Wire Wire Line
-	9250 4850 9250 4950
-Connection ~ 9250 5150
-Connection ~ 9250 4950
-Wire Wire Line
-	9250 4950 9250 5050
-Connection ~ 9250 5050
-Wire Wire Line
-	9250 5050 9250 5150
 Wire Wire Line
 	4950 5050 4650 5050
@@
 	1    0    0    -1
 $EndComp
-NoConn ~ 9250 2750
-NoConn ~ 9250 2850
-NoConn ~ 9250 3050
-NoConn ~ 9250 3150
-NoConn ~ 9250 3350
-NoConn ~ 9250 3550
+$Comp
+L Connector_Generic:Conn_02x04_Counter_Clockwise J2
+U 1 1 5FC55B49
+P 1150 6550
+F 0 "J2" H 1200 6867 50  0000 C CNN
+F 1 "Conn_02x04_Counter_Clockwise" H 1200 6776 50  0000 C CNN
+F 2 "footprints:SOIC_clipProgSmall" H 1150 6550 50  0001 C CNN
+F 3 "~" H 1150 6550 50  0001 C CNN
+	1    1150 6550
+	1    0    0    -1
+$EndComp
+Wire Wire Line
+	9250 4150 9250 4250
+Connection ~ 9250 4150
+Connection ~ 9250 4250
+Wire Wire Line
+	9250 4050 9250 4150
+Wire Wire Line
+	9250 3950 9250 4050
+Connection ~ 9250 4050
+Wire Wire Line
+	9250 4850 9250 4950
+Connection ~ 9250 4950
+Wire Wire Line
+	9250 5050 9250 5150
+Wire Wire Line
+	9250 4950 9250 5050
+Connection ~ 9250 5050
+Connection ~ 9250 5150
+$Comp
+L business-card-rescue:F1C100s-3340_kicad-business-card-rescue U7
+U 1 1 5FC1F3CA
+P 7050 3250
+F 0 "U7" H 7100 5415 50  0000 C CNN
+F 1 "F1C100s" H 7100 5324 50  0000 C CNN
+F 2 "footprints:QFN-88_EP_10x10_Pitch0.4mm" H 4950 4950 50  0001 C CNN
+F 3 "" H 4950 4950 50  0001 C CNN
+	1    7050 3250
+	1    0    0    -1
+$EndComp
+Wire Wire Line
+	9250 3050 9450 3050
+Wire Wire Line
+	9250 3150 9450 3150
+Wire Wire Line
+	9250 3350 9450 3350
+Wire Wire Line
+	9250 3550 9450 3550
+Text Label 9450 3050 0    50   ~ 0
+JTAG_TMS
+Text Label 9450 3150 0    50   ~ 0
+JTAG_TDI
+Text Label 9450 3350 0    50   ~ 0
+JTAG_TMS
+Text Label 9450 3550 0    50   ~ 0
+JTAG_TCK
+Text Label 9250 2750 0    50   ~ 0
+SCL
+Text Label 9250 2850 0    50   ~ 0
+SDA
+Wire Wire Line
+	1450 6450 1550 6450
+Wire Wire Line
+	1450 6550 1550 6550
+Wire Wire Line
+	1450 6650 1550 6650
+Wire Wire Line
+	1450 6750 1550 6750
+Wire Wire Line
+	950  6450 850  6450
+Wire Wire Line
+	950  6550 850  6550
+Wire Wire Line
+	950  6650 850  6650
+Wire Wire Line
+	950  6750 850  6750
+Text Label 1550 6450 0    50   ~ 0
+SDA
+Text Label 1550 6550 0    50   ~ 0
+JTAG_TDI
+Text Label 1550 6650 0    50   ~ 0
+JTAG_TCK
+Text Label 850  6450 2    50   ~ 0
+SCL
+Text Label 850  6550 2    50   ~ 0
+JTAG_TMS
+Text Label 850  6650 2    50   ~ 0
+JTAG_TDO
+NoConn ~ 850  6750
+$Comp
+L power:GND #PWR?
+U 1 1 5FC8A829
+P 1550 6750
+F 0 "#PWR?" H 1550 6500 50  0001 C CNN
+F 1 "GND" H 1555 6577 50  0000 C CNN
+F 2 "" H 1550 6750 50  0001 C CNN
+F 3 "" H 1550 6750 50  0001 C CNN
+	1    1550 6750
+	1    0    0    -1
+$EndComp
 $EndSCHEMATC

Commit message: images.
Parts:
- removed J2: Conn_02x04_Counter_Clockwise, footprints:SOIC_clipProgSmall, symbol Connector_Generic:Conn_02x04_Counter_Clockwise
- C7: footprint Capacitor_SMD:C_0805_2012Metric_Pad1.15x1.40mm_HandSolder -> Capacitor_SMD:C_0805_2012Metric_Pad1.18x1.45mm_HandSolder
- F1: footprint Fuse:Fuse_1812_4532Metric_Pad1.30x3.40mm_HandSolder -> Fuse:Fuse_0805_2012Metric
Connections:
- net JTAG_TCK: no longer names the net of U7.53 (PF5/SDC0_D2/DBG_CK/PWM1/EINTF5)
- net JTAG_TDI: no longer names the net of U7.57 (PF1/SDC0_D0/DBG_DI/EINTF1)
- net JTAG_TMS: no longer names the net of U7.55 (PF3/SDC0_CMD/DBG_DO/EINTF3)
- net JTAG_TMS: no longer U7.58 (PF0/SDC0_D1/DBG_MS/IR_RX/EINTF0)
- net SCL: no longer names the net of U7.38 (PE11/CLK_OUT/TWI0_SCK/IR_RX/EINTE11)
- net SDA: no longer names the net of U7.37 (PE12/DA_MCLK/TWI0_SDA/PWM0/EINTE12)
- no-connect marks 44 -> 49
Changed lines of the file:
@@
 EESchema Schematic File Version 4
-LIBS:business-card-cache
-EELAYER 26 0
+EELAYER 30 0
 EELAYER END
 $Descr A4 11693 8268
@@
 F 0 "F1" V 1500 500 50  0000 C CNN
 F 1 "Polyfuse" V 1500 750 50  0000 C CNN
-F 2 "Fuse:Fuse_1812_4532Metric_Pad1.30x3.40mm_HandSolder" H 1700 550 50  0001 L CNN
+F 2 "Fuse:Fuse_0805_2012Metric" H 1700 550 50  0001 L CNN
 F 3 "~" H 1650 750 50  0001 C CNN
 F 4 "R" H 1650 750 50  0001 C CNN "Spice_Primitive"
@@
 F 0 "C7" V 1250 4050 50  0000 C CNN
 F 1 "2u2" V 1250 4250 50  0000 C CNN
-F 2 "Capacitor_SMD:C_0805_2012Metric_Pad1.15x1.40mm_HandSolder" H 1250 4700 50  0001 C CNN
+F 2 "Capacitor_SMD:C_0805_2012Metric_Pad1.18x1.45mm_HandSolder" H 1250 4700 50  0001 C CNN
 F 3 "~" H 1250 4700 50  0001 C CNN
 	1    1250 4700
@@
 	1    0    0    -1
 $EndComp
-$Comp
-L Connector_Generic:Conn_02x04_Counter_Clockwise J2
-U 1 1 5FC55B49
-P 1150 6550
-F 0 "J2" H 1200 6867 50  0000 C CNN
-F 1 "Conn_02x04_Counter_Clockwise" H 1200 6776 50  0000 C CNN
-F 2 "footprints:SOIC_clipProgSmall" H 1150 6550 50  0001 C CNN
-F 3 "~" H 1150 6550 50  0001 C CNN
-	1    1150 6550
-	1    0    0    -1
-$EndComp
 Wire Wire Line
 	9250 4150 9250 4250
@@
 	1    0    0    -1
 $EndComp
-Wire Wire Line
-	9250 3050 9450 3050
-Wire Wire Line
-	9250 3150 9450 3150
-Wire Wire Line
-	9250 3350 9450 3350
-Wire Wire Line
-	9250 3550 9450 3550
-Text Label 9450 3050 0    50   ~ 0
-JTAG_TMS
-Text Label 9450 3150 0    50   ~ 0
-JTAG_TDI
-Text Label 9450 3350 0    50   ~ 0
-JTAG_TMS
-Text Label 9450 3550 0    50   ~ 0
-JTAG_TCK
-Text Label 9250 2750 0    50   ~ 0
-SCL
-Text Label 9250 2850 0    50   ~ 0
-SDA
-Wire Wire Line
-	1450 6450 1550 6450
-Wire Wire Line
-	1450 6550 1550 6550
-Wire Wire Line
-	1450 6650 1550 6650
-Wire Wire Line
-	1450 6750 1550 6750
-Wire Wire Line
-	950  6450 850  6450
-Wire Wire Line
-	950  6550 850  6550
-Wire Wire Line
-	950  6650 850  6650
-Wire Wire Line
-	950  6750 850  6750
-Text Label 1550 6450 0    50   ~ 0
-SDA
-Text Label 1550 6550 0    50   ~ 0
-JTAG_TDI
-Text Label 1550 6650 0    50   ~ 0
-JTAG_TCK
-Text Label 850  6450 2    50   ~ 0
-SCL
-Text Label 850  6550 2    50   ~ 0
-JTAG_TMS
-Text Label 850  6650 2    50   ~ 0
-JTAG_TDO
-NoConn ~ 850  6750
-$Comp
-L power:GND #PWR?
-U 1 1 5FC8A829
-P 1550 6750
-F 0 "#PWR?" H 1550 6500 50  0001 C CNN
-F 1 "GND" H 1555 6577 50  0000 C CNN
-F 2 "" H 1550 6750 50  0001 C CNN
-F 3 "" H 1550 6750 50  0001 C CNN
-	1    1550 6750
-	1    0    0    -1
-$EndComp
+NoConn ~ 9250 3050
+NoConn ~ 9250 3150
+NoConn ~ 9250 3350
+NoConn ~ 9250 3550
+NoConn ~ 9250 2750
+NoConn ~ 9250 2850
 $EndSCHEMATC
